File: RPiHAT/rpihat.sch (EAGLE design)
At the start: 37 parts

Commit message: Licensing
added License for the EEPROM design and CC4.0 BY-SA for Netz39 to the board.
Other:
- note added: "Designed by Andreas Watterott (Watterott electronic)"
- note added: "Released under the Creative Commons Attribution Share-Alike License"
- note added: "http://creativecommons.org/licenses/by-sa/4.0/"
Changed lines of the file:
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@@
 <grid distance="0.1" unitdist="inch" unit="inch" style="lines" multiple="1" display="no" altdistance="0.01" altunitdist="inch" altunit="inch"/>
 <layers>
-<layer number="1" name="Top" color="4" fill="1" visible="yes" active="no"/>
-<layer number="16" name="Bottom" color="1" fill="1" visible="yes" active="no"/>
-<layer number="17" name="Pads" color="2" fill="1" visible="yes" active="no"/>
-<layer number="18" name="Vias" color="2" fill="1" visible="yes" active="no"/>
-<layer number="19" name="Unrouted" color="6" fill="1" visible="yes" active="no"/>
-<layer number="20" name="Dimension" color="15" fill="1" visible="yes" active="no"/>
-<layer number="21" name="tPlace" color="7" fill="1" visible="yes" active="no"/>
-<layer number="22" name="bPlace" color="7" fill="1" visible="yes" active="no"/>
-<layer number="23" name="tOrigins" color="15" fill="1" visible="yes" active="no"/>
-<layer number="24" name="bOrigins" color="15" fill="1" visible="yes" active="no"/>
-<layer number="25" name="tNames" color="7" fill="1" visible="yes" active="no"/>
-<layer number="26" name="bNames" color="7" fill="1" visible="yes" active="no"/>
-<layer number="27" name="tValues" color="7" fill="1" visible="yes" active="no"/>
-<layer number="28" name="bValues" color="7" fill="1" visible="yes" active="no"/>
+<layer number="1" name="Top" color="4" fill="1" visible="no" active="no"/>
+<layer number="16" name="Bottom" color="1" fill="1" visible="no" active="no"/>
+<layer number="17" name="Pads" color="2" fill="1" visible="no" active="no"/>
+<layer number="18" name="Vias" color="2" fill="1" visible="no" active="no"/>
+<layer number="19" name="Unrouted" color="6" fill="1" visible="no" active="no"/>
+<layer number="20" name="Dimension" color="15" fill="1" visible="no" active="no"/>
+<layer number="21" name="tPlace" color="7" fill="1" visible="no" active="no"/>
+<layer number="22" name="bPlace" color="7" fill="1" visible="no" active="no"/>
+<layer number="23" name="tOrigins" color="15" fill="1" visible="no" active="no"/>
+<layer number="24" name="bOrigins" color="15" fill="1" visible="no" active="no"/>
+<layer number="25" name="tNames" color="7" fill="1" visible="no" active="no"/>
+<layer number="26" name="bNames" color="7" fill="1" visible="no" active="no"/>
+<layer number="27" name="tValues" color="7" fill="1" visible="no" active="no"/>
+<layer number="28" name="bValues" color="7" fill="1" visible="no" active="no"/>
 <layer number="29" name="tStop" color="7" fill="3" visible="no" active="no"/>
 <layer number="30" name="bStop" color="7" fill="6" visible="no" active="no"/>
@@
 <layer number="35" name="tGlue" color="7" fill="4" visible="no" active="no"/>
 <layer number="36" name="bGlue" color="7" fill="5" visible="no" active="no"/>
-<layer number="37" name="tTest" color="7" fill="1" visible="yes" active="no"/>
-<layer number="38" name="bTest" color="7" fill="1" visible="yes" active="no"/>
+<layer number="37" name="tTest" color="7" fill="1" visible="no" active="no"/>
+<layer number="38" name="bTest" color="7" fill="1" visible="no" active="no"/>
 <layer number="39" name="tKeepout" color="4" fill="11" visible="no" active="no"/>
 <layer number="40" name="bKeepout" color="1" fill="11" visible="no" active="no"/>
@@
 <layer number="44" name="Drills" color="7" fill="1" visible="no" active="no"/>
 <layer number="45" name="Holes" color="7" fill="1" visible="no" active="no"/>
-<layer number="46" name="Milling" color="3" fill="1" visible="yes" active="no"/>
-<layer number="47" name="Measures" color="7" fill="1" visible="yes" active="no"/>
-<layer number="48" name="Document" color="7" fill="1" visible="yes" active="no"/>
-<layer number="49" name="Reference" color="7" fill="1" visible="yes" active="no"/>
-<layer number="50" name="dxf" color="7" fill="1" visible="yes" active="no"/>
-<layer number="51" name="tDocu" color="7" fill="1" visible="yes" active="no"/>
-<layer number="52" name="bDocu" color="7" fill="1" visible="yes" active="no"/>
-<layer number="53" name="tCopper" color="7" fill="11" visible="yes" active="no"/>
-<layer number="54" name="bCopper" color="7" fill="1" visible="yes" active="no"/>
-<layer number="56" name="wert" color="7" fill="1" visible="yes" active="no"/>
-<layer number="57" name="tCAD" color="7" fill="1" visible="yes" active="no"/>
+<layer number="46" name="Milling" color="3" fill="1" visible="no" active="no"/>
+<layer number="47" name="Measures" color="7" fill="1" visible="no" active="no"/>
+<layer number="48" name="Document" color="7" fill="1" visible="no" active="no"/>
+<layer number="49" name="Reference" color="7" fill="1" visible="no" active="no"/>
+<layer number="50" name="dxf" color="7" fill="1" visible="no" active="no"/>
+<layer number="51" name="tDocu" color="7" fill="1" visible="no" active="no"/>
+<layer number="52" name="bDocu" color="7" fill="1" visible="no" active="no"/>
+<layer number="53" name="tCopper" color="7" fill="11" visible="no" active="no"/>
+<layer number="54" name="bCopper" color="7" fill="1" visible="no" active="no"/>
+<layer number="56" name="wert" color="7" fill="1" visible="no" active="no"/>
+<layer number="57" name="tCAD" color="7" fill="1" visible="no" active="no"/>
 <layer number="90" name="Modules" color="5" fill="1" visible="yes" active="yes"/>
 <layer number="91" name="Nets" color="2" fill="1" visible="yes" active="yes"/>
@@
 <wire x1="104.14" y1="66.04" x2="104.14" y2="137.16" width="0.1524" layer="97"/>
 <text x="106.68" y="134.62" size="1.778" layer="97">Testpoints</text>
+<text x="10.16" y="55.88" size="1.778" layer="97">Designed by Andreas Watterott (Watterott electronic)</text>
+<text x="106.68" y="53.34" size="1.778" layer="97">http://creativecommons.org/licenses/by-sa/4.0/</text>
+<text x="106.68" y="55.88" size="1.778" layer="97">Released under the Creative Commons Attribution Share-Alike License</text>
 </plain>
 <instances>

Commit message: RPi HAT: Documentation
Parts:
- renumbered IC to U1
Changed lines of the file:
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@@
 <part name="R2" library="we-rcl" deviceset="RESISTOR" device="-R0603" value="3k9"/>
 <part name="R3" library="we-rcl" deviceset="RESISTOR" device="-R0603" value="3k9"/>
-<part name="IC" library="we-chip" deviceset="24LC*" device="-I/OT"/>
+<part name="U1" library="we-chip" deviceset="24LC*" device="-I/OT"/>
 <part name="GPIO06" library="testpad" deviceset="PTR1" device="TP06R" value="PTR1TP06R"/>
 <part name="GPIO13" library="testpad" deviceset="PTR1" device="TP06R" value="PTR1TP06R"/>
@@
 <instance part="R2" gate="R" x="72.39" y="27.94" rot="R90"/>
 <instance part="R3" gate="R" x="31.75" y="24.13" rot="R90"/>
-<instance part="IC" gate="IC" x="49.53" y="22.86"/>
+<instance part="U1" gate="IC" x="49.53" y="22.86"/>
 <instance part="GPIO06" gate="G$1" x="175.26" y="109.22" smashed="yes" rot="R270">
 <attribute name="NAME" x="160.02" y="108.966" size="1.778" layer="95"/>
@@
 <pinref part="GND2" gate="1" pin="GND"/>
 <wire x1="74.93" y1="17.78" x2="67.31" y2="17.78" width="0.1524" layer="91"/>
-<pinref part="IC" gate="IC" pin="GND"/>
+<pinref part="U1" gate="IC" pin="GND"/>
 </segment>
 <segment>
@@
 <junction x="67.31" y="33.02"/>
 <pinref part="R2" gate="R" pin="2"/>
-<pinref part="IC" gate="IC" pin="VCC"/>
+<pinref part="U1" gate="IC" pin="VCC"/>
 </segment>
 <segment>
@@
 <wire x1="72.39" y1="22.86" x2="67.31" y2="22.86" width="0.1524" layer="91"/>
 <junction x="72.39" y="22.86"/>
-<pinref part="IC" gate="IC" pin="SDA"/>
+<pinref part="U1" gate="IC" pin="SDA"/>
 </segment>
 <segment>
@@
 <wire x1="24.13" y1="22.86" x2="34.29" y2="22.86" width="0.1524" layer="91"/>
 <junction x="24.13" y="22.86"/>
-<pinref part="IC" gate="IC" pin="SCL"/>
+<pinref part="U1" gate="IC" pin="SCL"/>
 </segment>
 <segment>
@@
 <pinref part="WP" gate="J" pin="2"/>
 <pinref part="R3" gate="R" pin="1"/>
-<pinref part="IC" gate="IC" pin="WP"/>
-</segment>
-</net>
+<pinref part="U1" gate="IC" pin="WP"/>
+</segment>
+</net>
